Commit message: add collision elements to urdf

File: urdf/sektion_cabinet.urdf (robot description, URDF)
Before this commit: robot cabinet_sektion, 15 links, 14 joints
Links:
- link door_left_link: geometry collision mesh filename=package://sektion_cabinet_model/meshes/door_left.stl scale=1.0 1.0 1.0; visual mesh filename=package://sektion_cabinet_model/meshes/door_left.stl scale=1.0 1.0 1.0
- link door_left_nob_link: geometry collision mesh filename=package://sektion_cabinet_model/meshes/door_left_nob.stl scale=1.0 1.0 1.0; visual mesh filename=package://sektion_cabinet_model/meshes/door_left_nob.stl scale=1.0 1.0 1.0
- link door_right_link: geometry collision mesh filename=package://sektion_cabinet_model/meshes/door_right.stl scale=1.0 1.0 1.0; visual mesh filename=package://sektion_cabinet_model/meshes/door_right.stl scale=1.0 1.0 1.0
- link door_right_nob_link: geometry collision mesh filename=package://sektion_cabinet_model/meshes/door_right_nob.stl scale=1.0 1.0 1.0; visual mesh filename=package://sektion_cabinet_model/meshes/door_right_nob.stl scale=1.0 1.0 1.0
- link drawer_bottom: geometry collision mesh filename=package://sektion_cabinet_model/meshes/drawer.stl scale=1.0 1.0 1.0; visual mesh filename=package://sektion_cabinet_model/meshes/drawer.stl scale=1.0 1.0 1.0
- link drawer_handle_bottom: geometry collision mesh filename=package://sektion_cabinet_model/meshes/drawer_handle.stl scale=1.0 1.0 1.0; visual mesh filename=package://sektion_cabinet_model/meshes/drawer_handle.stl scale=1.0 1.0 1.0
- link drawer_handle_top: geometry collision mesh filename=package://sektion_cabinet_model/meshes/drawer_handle.stl scale=1.0 1.0 1.0; visual mesh filename=package://sektion_cabinet_model/meshes/drawer_handle.stl scale=1.0 1.0 1.0
- link drawer_top: geometry collision mesh filename=package://sektion_cabinet_model/meshes/drawer.stl scale=1.0 1.0 1.0; visual mesh filename=package://sektion_cabinet_model/meshes/drawer.stl scale=1.0 1.0 1.0
- link sektion: geometry collision mesh filename=package://sektion_cabinet_model/meshes/sektion.stl scale=1.0 1.0 1.0; visual mesh filename=package://sektion_cabinet_model/meshes/sektion.stl scale=1.0 1.0 1.0

Commit message: update again

File: urdf/sektion_cabinet.urdf (robot description, URDF)
Before this commit: robot cabinet_sektion, 15 links, 14 joints
Links:
- link door_left_anchor_link: mass None -> 0.001
- link door_left_joint_anchor_link: mass None -> 0.001
- link door_right_anchor_link: mass None -> 0.001
- link door_right_joint_anchor_link: mass None -> 0.001
